Commit message: gazebo publishes ros2 topics properly

File: src/leo_rover_description/urdf/leo_rover_with_sensors.urdf.xacro (robot description, xacro)
@@ -1,41 +1,87 @@
 <?xml version="1.0"?>
 <robot xmlns:xacro="http://www.ros.org/wiki/xacro" name="leo_rover">
-  <!-- REQUIRED ARGUMENT -->
+  <!-- Expose the namespace argument so the launch file can pass "leo1", "leo2", etc. -->
   <xacro:arg name="robot_ns" default="leo"/>
-  <!-- Base Leo model -->
+  <!-- Include the base Leo Rover macro -->
   <xacro:include filename="$(find leo_description)/urdf/leo_sim.urdf.xacro"/>
-  <!-- LiDAR -->
-  <gazebo reference="base_link">
-    <sensor name="lidar" type="gpu_lidar">
+  <!-- ================= SENSOR LINKS & JOINTS ================= -->
+  <!-- Simplified dummy links with minimal inertia for Gazebo physics stability -->
+  <link name="sensor_lidar_link">
+    <inertial>
+      <mass value="0.1"/>
+      <inertia ixx="0.001" ixy="0" ixz="0" iyy="0.001" iyz="0" izz="0.001"/>
+    </inertial>
+  </link>
+  <joint name="sensor_lidar_joint" type="fixed">
+    <parent link="$(arg robot_ns)/base_link"/>
+    <child link="sensor_lidar_link"/>
+    <origin xyz="0.2 0 0.4" rpy="0 0 0"/>
+  </joint>
+  <link name="sensor_camera_link">
+    <inertial>
+      <mass value="0.05"/>
+      <inertia ixx="0.0001" ixy="0" ixz="0" iyy="0.0001" iyz="0" izz="0.0001"/>
+    </inertial>
+  </link>
+  <joint name="sensor_camera_joint" type="fixed">
+    <parent link="$(arg robot_ns)/base_link"/>
+    <child link="sensor_camera_link"/>
+    <origin xyz="0.25 0 0.2" rpy="0 0 0"/>
+  </joint>
+  <link name="sensor_imu_link">
+    <inertial>
+      <mass value="0.01"/>
+      <inertia ixx="0.00001" ixy="0" ixz="0" iyy="0.00001" iyz="0" izz="0.00001"/>
+    </inertial>
+  </link>
+  <joint name="sensor_imu_joint" type="fixed">
+    <parent link="$(arg robot_ns)/base_link"/>
+    <child link="sensor_imu_link"/>
+    <origin xyz="0 0 0.1" rpy="0 0 0"/>
+  </joint>
+  <!-- ================= GAZEBO SENSOR CONFIGURATIONS ================= -->
+  <!-- 3D LiDAR -->
+  <gazebo reference="sensor_lidar_link">
+    <sensor name="gpu_lidar" type="gpu_lidar">
+      <always_on>true</always_on>
+      <visualize>true</visualize>
       <update_rate>10</update_rate>
+      <!-- Namespaced Topic -->
       <topic>/$(arg robot_ns)/scan</topic>
-      <gz>
-        <frame_id>$(arg robot_ns)/base_link</frame_id>
-      </gz>
-      <ray>
+      <!-- Namespaced TF Frame -->
+      <gz_frame_id>$(arg robot_ns)/sensor_lidar_link</gz_frame_id>
+      <lidar>
         <scan>
           <horizontal>
             <samples>720</samples>
+            <resolution>1</resolution>
             <min_angle>-3.14159</min_angle>
             <max_angle>3.14159</max_angle>
           </horizontal>
+          <vertical>
+            <samples>16</samples>
+            <resolution>1</resolution>
+            <min_angle>-0.26</min_angle>
+            <max_angle>0.26</max_angle>
+          </vertical>
         </scan>
         <range>
-          <min>0.05</min>
-          <max>12.0</max>
+          <min>0.1</min>
+          <max>20.0</max>
+          <resolution>0.01</resolution>
         </range>
-      </ray>
-      <always_on>1</always_on>
-      <visualize>true</visualize>
+      </lidar>
+      <point_cloud>true</point_cloud>
     </sensor>
   </gazebo>
-  <!-- Camera -->
-  <gazebo reference="camera_frame">
+  <!-- RGBD Camera -->
+  <gazebo reference="sensor_camera_link">
     <sensor name="rgbd_camera" type="rgbd_camera">
+      <always_on>true</always_on>
       <update_rate>30</update_rate>
+      <!-- Namespaced Topic -->
       <topic>/$(arg robot_ns)/camera</topic>
-      <gz>
-        <frame_id>$(arg robot_ns)/camera_frame</frame_id>
-      </gz>
+      <!-- Namespaced TF Frame -->
+      <gz_frame_id>$(arg robot_ns)/sensor_camera_link</gz_frame_id>
       <camera>
         <horizontal_fov>1.047</horizontal_fov>
@@ -43,24 +89,23 @@
           <width>640</width>
           <height>480</height>
+          <format>R8G8B8</format>
         </image>
-        <depth_camera>
-          <clip>
-            <near>0.1</near>
-            <far>10.0</far>
-          </clip>
-        </depth_camera>
+        <clip>
+          <near>0.1</near>
+          <far>10.0</far>
+        </clip>
       </camera>
-      <always_on>1</always_on>
     </sensor>
   </gazebo>
   <!-- IMU -->
-  <gazebo reference="base_link">
-    <sensor name="leo_imu_sensor" type="imu">
-      <always_on>1</always_on>
+  <gazebo reference="sensor_imu_link">
+    <sensor name="imu_sensor" type="imu">
+      <always_on>true</always_on>
       <update_rate>100</update_rate>
-      <topic>/$(arg robot_ns)/imu</topic>
-      <gz>
-        <frame_id>$(arg robot_ns)/base_link</frame_id>
-      </gz>
+      <!-- Namespaced Topic -->
+      <topic>/$(arg robot_ns)/imu/data</topic>
+      <!-- Namespaced TF Frame -->
+      <gz_frame_id>$(arg robot_ns)/sensor_imu_link</gz_frame_id>
+      <imu/>
     </sensor>
   </gazebo>

Commit message: fixed rviz2.

File: src/leo_rover_description/urdf/leo_rover_with_sensors.urdf.xacro (robot description, xacro)
@@ -1,13 +1,11 @@
 <?xml version="1.0"?>
 <robot xmlns:xacro="http://www.ros.org/wiki/xacro" name="leo_rover">
-  <!-- Expose the namespace argument so the launch file can pass "leo1", "leo2", etc. -->
   <xacro:arg name="robot_ns" default="leo"/>
-  <!-- Include the base Leo Rover macro -->
   <xacro:include filename="$(find leo_description)/urdf/leo_sim.urdf.xacro"/>
   <!-- ================= SENSOR LINKS & JOINTS ================= -->
-  <!-- Simplified dummy links with minimal inertia for Gazebo physics stability -->
-  <link name="sensor_lidar_link">
+  <link name="$(arg robot_ns)/sensor_lidar_link">
     <inertial>
       <mass value="0.1"/>
+      <origin xyz="0 0 0"/>
       <inertia ixx="0.001" ixy="0" ixz="0" iyy="0.001" iyz="0" izz="0.001"/>
     </inertial>
@@ -15,10 +13,11 @@
   <joint name="sensor_lidar_joint" type="fixed">
     <parent link="$(arg robot_ns)/base_link"/>
-    <child link="sensor_lidar_link"/>
+    <child link="$(arg robot_ns)/sensor_lidar_link"/>
     <origin xyz="0.2 0 0.4" rpy="0 0 0"/>
   </joint>
-  <link name="sensor_camera_link">
+  <link name="$(arg robot_ns)/sensor_camera_link">
     <inertial>
       <mass value="0.05"/>
+      <origin xyz="0 0 0"/>
       <inertia ixx="0.0001" ixy="0" ixz="0" iyy="0.0001" iyz="0" izz="0.0001"/>
     </inertial>
@@ -26,10 +25,11 @@
   <joint name="sensor_camera_joint" type="fixed">
     <parent link="$(arg robot_ns)/base_link"/>
-    <child link="sensor_camera_link"/>
+    <child link="$(arg robot_ns)/sensor_camera_link"/>
     <origin xyz="0.25 0 0.2" rpy="0 0 0"/>
   </joint>
-  <link name="sensor_imu_link">
+  <link name="$(arg robot_ns)/sensor_imu_link">
     <inertial>
       <mass value="0.01"/>
+      <origin xyz="0 0 0"/>
       <inertia ixx="0.00001" ixy="0" ixz="0" iyy="0.00001" iyz="0" izz="0.00001"/>
     </inertial>
@@ -37,17 +37,14 @@
   <joint name="sensor_imu_joint" type="fixed">
     <parent link="$(arg robot_ns)/base_link"/>
-    <child link="sensor_imu_link"/>
+    <child link="$(arg robot_ns)/sensor_imu_link"/>
     <origin xyz="0 0 0.1" rpy="0 0 0"/>
   </joint>
   <!-- ================= GAZEBO SENSOR CONFIGURATIONS ================= -->
-  <!-- 3D LiDAR -->
-  <gazebo reference="sensor_lidar_link">
+  <gazebo reference="$(arg robot_ns)/sensor_lidar_link">
     <sensor name="gpu_lidar" type="gpu_lidar">
       <always_on>true</always_on>
       <visualize>true</visualize>
       <update_rate>10</update_rate>
-      <!-- Namespaced Topic -->
       <topic>/$(arg robot_ns)/scan</topic>
-      <!-- Namespaced TF Frame -->
       <gz_frame_id>$(arg robot_ns)/sensor_lidar_link</gz_frame_id>
       <lidar>
@@ -75,12 +72,9 @@
     </sensor>
   </gazebo>
-  <!-- RGBD Camera -->
-  <gazebo reference="sensor_camera_link">
+  <gazebo reference="$(arg robot_ns)/sensor_camera_link">
     <sensor name="rgbd_camera" type="rgbd_camera">
       <always_on>true</always_on>
       <update_rate>30</update_rate>
-      <!-- Namespaced Topic -->
       <topic>/$(arg robot_ns)/camera</topic>
-      <!-- Namespaced TF Frame -->
       <gz_frame_id>$(arg robot_ns)/sensor_camera_link</gz_frame_id>
       <camera>
@@ -98,12 +92,9 @@
     </sensor>
   </gazebo>
-  <!-- IMU -->
-  <gazebo reference="sensor_imu_link">
+  <gazebo reference="$(arg robot_ns)/sensor_imu_link">
     <sensor name="imu_sensor" type="imu">
       <always_on>true</always_on>
       <update_rate>100</update_rate>
-      <!-- Namespaced Topic -->
       <topic>/$(arg robot_ns)/imu/data</topic>
-      <!-- Namespaced TF Frame -->
       <gz_frame_id>$(arg robot_ns)/sensor_imu_link</gz_frame_id>
       <imu/>

Commit message: Added docker container to develop in ROS2 Humble.

File: src/leo_rover_description/urdf/leo_rover_with_sensors.urdf.xacro (robot description, xacro)
@@ -2,16 +2,25 @@
 <robot xmlns:xacro="http://www.ros.org/wiki/xacro" name="leo_rover">
   <xacro:arg name="robot_ns" default="leo"/>
-  <xacro:include filename="$(find leo_description)/urdf/leo_sim.urdf.xacro"/>
-  <!-- ================= SENSOR LINKS & JOINTS ================= -->
+  <!--
+    Use leo.urdf.xacro (base robot: links, joints, meshes, inertia) instead of
+    leo_sim.urdf.xacro, which was written for Gazebo Ignition/Fortress and
+    references the deprecated ros_ign_sim package, causing launch failures on
+    Gazebo Harmonic.  All Gazebo Harmonic plugins are defined below.
+  -->
+  <xacro:include filename="$(find leo_description)/urdf/leo.urdf.xacro"/>
+  <!-- ================================================================== -->
+  <!-- Sensor links & joints                                               -->
+  <!-- ================================================================== -->
   <link name="$(arg robot_ns)/sensor_lidar_link">
     <inertial>
       <mass value="0.1"/>
       <origin xyz="0 0 0"/>
-      <inertia ixx="0.001" ixy="0" ixz="0" iyy="0.001" iyz="0" izz="0.001"/>
+      <inertia ixx="0.001" ixy="0" ixz="0"
+               iyy="0.001" iyz="0" izz="0.001"/>
     </inertial>
   </link>
   <joint name="sensor_lidar_joint" type="fixed">
     <parent link="$(arg robot_ns)/base_link"/>
-    <child link="$(arg robot_ns)/sensor_lidar_link"/>
+    <child  link="$(arg robot_ns)/sensor_lidar_link"/>
     <origin xyz="0.2 0 0.4" rpy="0 0 0"/>
   </joint>
@@ -20,10 +29,11 @@
       <mass value="0.05"/>
       <origin xyz="0 0 0"/>
-      <inertia ixx="0.0001" ixy="0" ixz="0" iyy="0.0001" iyz="0" izz="0.0001"/>
+      <inertia ixx="0.0001" ixy="0" ixz="0"
+               iyy="0.0001" iyz="0" izz="0.0001"/>
     </inertial>
   </link>
   <joint name="sensor_camera_joint" type="fixed">
     <parent link="$(arg robot_ns)/base_link"/>
-    <child link="$(arg robot_ns)/sensor_camera_link"/>
+    <child  link="$(arg robot_ns)/sensor_camera_link"/>
     <origin xyz="0.25 0 0.2" rpy="0 0 0"/>
   </joint>
@@ -32,13 +42,51 @@
       <mass value="0.01"/>
       <origin xyz="0 0 0"/>
-      <inertia ixx="0.00001" ixy="0" ixz="0" iyy="0.00001" iyz="0" izz="0.00001"/>
+      <inertia ixx="0.00001" ixy="0" ixz="0"
+               iyy="0.00001" iyz="0" izz="0.00001"/>
     </inertial>
   </link>
   <joint name="sensor_imu_joint" type="fixed">
     <parent link="$(arg robot_ns)/base_link"/>
-    <child link="$(arg robot_ns)/sensor_imu_link"/>
+    <child  link="$(arg robot_ns)/sensor_imu_link"/>
     <origin xyz="0 0 0.1" rpy="0 0 0"/>
   </joint>
-  <!-- ================= GAZEBO SENSOR CONFIGURATIONS ================= -->
+  <!-- ================================================================== -->
+  <!-- Gazebo Harmonic — Differential Drive                                -->
+  <!--                                                                     -->
+  <!-- Leo Rover is a 4-wheel robot driven as two differential pairs.      -->
+  <!-- Joint names come from leo_description; verify with:                 -->
+  <!--   xacro $(find leo_description)/urdf/leo.urdf.xacro | grep joint   -->
+  <!-- ================================================================== -->
+  <gazebo>
+    <plugin filename="gz-sim-diff-drive-system"
+            name="gz::sim::systems::DiffDrive">
+      <left_joint>wheel_FL_joint</left_joint>
+      <left_joint>wheel_RL_joint</left_joint>
+      <right_joint>wheel_FR_joint</right_joint>
+      <right_joint>wheel_RR_joint</right_joint>
+      <!-- Leo Rover physical dimensions -->
+      <wheel_separation>0.358</wheel_separation>
+      <wheel_radius>0.0625</wheel_radius>
+      <!-- Namespaced topics so each robot is independent -->
+      <topic>/$(arg robot_ns)/cmd_vel</topic>
+      <odom_topic>/$(arg robot_ns)/odom</odom_topic>
+      <tf_topic>/$(arg robot_ns)/tf</tf_topic>
+      <frame_id>$(arg robot_ns)/odom</frame_id>
+      <child_frame_id>$(arg robot_ns)/base_link</child_frame_id>
+      <odom_publish_frequency>50</odom_publish_frequency>
+      <max_linear_velocity>1.0</max_linear_velocity>
+      <max_angular_velocity>2.0</max_angular_velocity>
+    </plugin>
+  </gazebo>
+  <!-- Publishes all wheel joint states so robot_state_publisher can work -->
+  <gazebo>
+    <plugin filename="gz-sim-joint-state-publisher-system"
+            name="gz::sim::systems::JointStatePublisher">
+      <topic>/$(arg robot_ns)/joint_states</topic>
+    </plugin>
+  </gazebo>
+  <!-- ================================================================== -->
+  <!-- Gazebo Harmonic — Sensors                                           -->
+  <!-- ================================================================== -->
   <gazebo reference="$(arg robot_ns)/sensor_lidar_link">
     <sensor name="gpu_lidar" type="gpu_lidar">

Commit message: changed tf topic mappings.

File: src/leo_rover_description/urdf/leo_rover_with_sensors.urdf.xacro (robot description, xacro)
@@ -2,20 +2,10 @@
 <robot xmlns:xacro="http://www.ros.org/wiki/xacro" name="leo_rover">
   <xacro:arg name="robot_ns" default="leo"/>
-  <!--
-    Use leo.urdf.xacro (base robot: links, joints, meshes, inertia) instead of
-    leo_sim.urdf.xacro, which was written for Gazebo Ignition/Fortress and
-    references the deprecated ros_ign_sim package, causing launch failures on
-    Gazebo Harmonic.  All Gazebo Harmonic plugins are defined below.
-  -->
   <xacro:include filename="$(find leo_description)/urdf/leo.urdf.xacro"/>
-  <!-- ================================================================== -->
-  <!-- Sensor links & joints                                               -->
-  <!-- ================================================================== -->
   <link name="$(arg robot_ns)/sensor_lidar_link">
     <inertial>
       <mass value="0.1"/>
       <origin xyz="0 0 0"/>
-      <inertia ixx="0.001" ixy="0" ixz="0"
-               iyy="0.001" iyz="0" izz="0.001"/>
+      <inertia ixx="0.001" ixy="0" ixz="0" iyy="0.001" iyz="0" izz="0.001"/>
     </inertial>
   </link>
@@ -29,6 +19,5 @@
       <mass value="0.05"/>
       <origin xyz="0 0 0"/>
-      <inertia ixx="0.0001" ixy="0" ixz="0"
-               iyy="0.0001" iyz="0" izz="0.0001"/>
+      <inertia ixx="0.0001" ixy="0" ixz="0" iyy="0.0001" iyz="0" izz="0.0001"/>
     </inertial>
   </link>
@@ -42,6 +31,5 @@
       <mass value="0.01"/>
       <origin xyz="0 0 0"/>
-      <inertia ixx="0.00001" ixy="0" ixz="0"
-               iyy="0.00001" iyz="0" izz="0.00001"/>
+      <inertia ixx="0.00001" ixy="0" ixz="0" iyy="0.00001" iyz="0" izz="0.00001"/>
     </inertial>
   </link>
@@ -51,42 +39,24 @@
     <origin xyz="0 0 0.1" rpy="0 0 0"/>
   </joint>
-  <!-- ================================================================== -->
-  <!-- Gazebo Harmonic — Differential Drive                                -->
-  <!--                                                                     -->
-  <!-- Leo Rover is a 4-wheel robot driven as two differential pairs.      -->
-  <!-- Joint names come from leo_description; verify with:                 -->
-  <!--   xacro $(find leo_description)/urdf/leo.urdf.xacro | grep joint   -->
-  <!-- ================================================================== -->
   <gazebo>
-    <plugin filename="gz-sim-diff-drive-system"
-            name="gz::sim::systems::DiffDrive">
+    <plugin filename="gz-sim-diff-drive-system" name="gz::sim::systems::DiffDrive">
       <left_joint>wheel_FL_joint</left_joint>
       <left_joint>wheel_RL_joint</left_joint>
       <right_joint>wheel_FR_joint</right_joint>
       <right_joint>wheel_RR_joint</right_joint>
-      <!-- Leo Rover physical dimensions -->
       <wheel_separation>0.358</wheel_separation>
       <wheel_radius>0.0625</wheel_radius>
-      <!-- Namespaced topics so each robot is independent -->
       <topic>/$(arg robot_ns)/cmd_vel</topic>
       <odom_topic>/$(arg robot_ns)/odom</odom_topic>
-      <tf_topic>/$(arg robot_ns)/tf</tf_topic>
-      <frame_id>$(arg robot_ns)/odom</frame_id>
-      <child_frame_id>$(arg robot_ns)/base_link</child_frame_id>
+      <frame_id>odom</frame_id>
+      <child_frame_id>base_link</child_frame_id>
       <odom_publish_frequency>50</odom_publish_frequency>
-      <max_linear_velocity>1.0</max_linear_velocity>
-      <max_angular_velocity>2.0</max_angular_velocity>
     </plugin>
   </gazebo>
-  <!-- Publishes all wheel joint states so robot_state_publisher can work -->
   <gazebo>
-    <plugin filename="gz-sim-joint-state-publisher-system"
-            name="gz::sim::systems::JointStatePublisher">
+    <plugin filename="gz-sim-joint-state-publisher-system" name="gz::sim::systems::JointStatePublisher">
       <topic>/$(arg robot_ns)/joint_states</topic>
     </plugin>
   </gazebo>
-  <!-- ================================================================== -->
-  <!-- Gazebo Harmonic — Sensors                                           -->
-  <!-- ================================================================== -->
   <gazebo reference="$(arg robot_ns)/sensor_lidar_link">
     <sensor name="gpu_lidar" type="gpu_lidar">
@@ -104,10 +74,4 @@
             <max_angle>3.14159</max_angle>
           </horizontal>
-          <vertical>
-            <samples>16</samples>
-            <resolution>1</resolution>
-            <min_angle>-0.26</min_angle>
-            <max_angle>0.26</max_angle>
-          </vertical>
         </scan>
         <range>
@@ -117,5 +81,4 @@
         </range>
       </lidar>
-      <point_cloud>true</point_cloud>
     </sensor>
   </gazebo>
@@ -133,8 +96,4 @@
           <format>R8G8B8</format>
         </image>
-        <clip>
-          <near>0.1</near>
-          <far>10.0</far>
-        </clip>
       </camera>
     </sensor>
